Commit message: added gazebo/moveit support

File: robot_craig_sim/urdf/robot_craig.xacro (robot description, xacro)
@@ -3,4 +3,6 @@
   <!-- Macros de links y joints generalizados -->
   <xacro:include filename="$(find robot_craig_sim)/urdf/robot_craig_joints.xacro"/>
+  <!-- Import all Gazebo-customization elements, including Gazebo colors -->
+  <xacro:include filename="$(find robot_craig_sim)/urdf/robot_craig.gazebo"/>
   <!-- LINKS -->
   <!-- base -->

File: robot_craig_sim/urdf/robot_craig_joints.xacro (robot description, xacro)
@@ -28,4 +28,14 @@
     <limit effort="1000" lower="-3.1416" upper="3.1416" velocity="2.618"/>
   </joint>
+	<transmission name="trans_joint_2">
+		<type>transmission_interface/SimpleTransmission</type>
+		<joint name="joint_2">
+			<hardwareInterface>hardware_interface/PositionJointInterface</hardwareInterface>
+		</joint>
+		<actuator name="motor_joint_2">
+			<hardwareInterface>hardware_interface/PositionJointInterface</hardwareInterface>
+			<mechanicalReduction>1</mechanicalReduction>
+		</actuator>
+  </transmission>
 	<!--joint3-->
 	<joint name="joint_3" type="revolute">
@@ -36,4 +46,14 @@
     <limit effort="1000" lower="-3.1416" upper="3.1416" velocity="2.618"/>
   </joint>
+	<transmission name="trans_joint_3">
+		<type>transmission_interface/SimpleTransmission</type>
+		<joint name="joint_3">
+			<hardwareInterface>hardware_interface/PositionJointInterface</hardwareInterface>
+		</joint>
+		<actuator name="motor_joint_3">
+			<hardwareInterface>hardware_interface/PositionJointInterface</hardwareInterface>
+			<mechanicalReduction>1</mechanicalReduction>
+		</actuator>
+  </transmission>
 	<!--joint4-->
 	<joint name="joint_4" type="revolute">
@@ -44,4 +64,14 @@
     <limit effort="1000" lower="-3.1416" upper="3.1416" velocity="2.618"/>
   </joint>
+	<transmission name="trans_joint_4">
+		<type>transmission_interface/SimpleTransmission</type>
+		<joint name="joint_4">
+			<hardwareInterface>hardware_interface/PositionJointInterface</hardwareInterface>
+		</joint>
+		<actuator name="motor_joint_4">
+			<hardwareInterface>hardware_interface/PositionJointInterface</hardwareInterface>
+			<mechanicalReduction>1</mechanicalReduction>
+		</actuator>
+  </transmission>
 	<!--joint5-->
 	<joint name="joint_5" type="revolute">
@@ -52,4 +82,14 @@
     <limit effort="1000" lower="-3.1416" upper="3.1416" velocity="2.618"/>
   </joint>
+	<transmission name="trans_joint_5">
+		<type>transmission_interface/SimpleTransmission</type>
+		<joint name="joint_5">
+			<hardwareInterface>hardware_interface/PositionJointInterface</hardwareInterface>
+		</joint>
+		<actuator name="motor_joint_5">
+			<hardwareInterface>hardware_interface/PositionJointInterface</hardwareInterface>
+			<mechanicalReduction>1</mechanicalReduction>
+		</actuator>
+  </transmission>
 	<!--joint6-->
 	<joint name="joint_6" type="revolute">
@@ -60,3 +100,13 @@
     <limit effort="1000" lower="-3.1416" upper="3.1416" velocity="2.618"/>
   </joint>
+	<transmission name="trans_joint_6">
+		<type>transmission_interface/SimpleTransmission</type>
+		<joint name="joint_6">
+			<hardwareInterface>hardware_interface/PositionJointInterface</hardwareInterface>
+		</joint>
+		<actuator name="motor_joint_6">
+			<hardwareInterface>hardware_interface/PositionJointInterface</hardwareInterface>
+			<mechanicalReduction>1</mechanicalReduction>
+		</actuator>
+  </transmission>
 </robot>
